File: ECAD/MainBoard-PAMI-2025/MainBoard-PAMI-2025.kicad_sch (KiCad schematic)
At the start: 65 parts, among them J1 Sensor_Center, J10 Serial, J11 Con_Batt, J13 OLED, J2 USB_B, J3 Sensor_RIGHT, J4 Servo, J5 Sensor_LEFT, J6 Servo, J7 LeftMotor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

Commit message: routage + silkscreen
Connections:
- net GPIOI_CENTER: no longer names the net of J1.5 (Pin_5)
- net GPIOI_LEFT: no longer names the net of J5.5 (Pin_5)
- net GPIOI_RIGHT: no longer names the net of J3.5 (Pin_5)
Changed lines of the file:
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@@
-	(wire
-		(pts
-			(xy 29.21 154.94) (xy 31.75 154.94)
-		)
-		(stroke
-			(width 0)
-			(type default)
-		)
-	)
 	(wire
 		(pts
@@
 	(wire
 		(pts
-			(xy 29.21 172.72) (xy 31.75 172.72)
-		)
-		(stroke
-			(width 0)
-			(type default)
-		)
-	)
-	(wire
-		(pts
 			(xy 41.91 46.99) (xy 41.91 48.26)
 		)
@@
 		(pts
 			(xy 276.86 82.55) (xy 271.78 82.55)
-		)
-		(stroke
-			(width 0)
-			(type default)
-		)
-	)
-	(wire
-		(pts
-			(xy 29.21 190.5) (xy 31.75 190.5)
 		)
 		(stroke
@@
 		)
 	)
-	(global_label "GPIOI_LEFT"
-		(shape input)
-		(at 29.21 190.5 180)
-		(fields_autoplaced yes)
-		(effects
-			(font
-				(size 1.27 1.27)
-			)
-			(justify right)
-		)
-		(property "Intersheetrefs" "${INTERSHEET_REFS}"
-			(at 15.9438 190.5 0)
-			(effects
-				(font
-					(size 1.27 1.27)
-				)
-				(justify right)
-				(hide yes)
-			)
-		)
-	)
 	(global_label "RightMS1"
 		(shape input)
@@
 		)
 	)
-	(global_label "GPIOI_RIGHT"
-		(shape input)
-		(at 29.21 154.94 180)
-		(fields_autoplaced yes)
-		(effects
-			(font
-				(size 1.27 1.27)
-			)
-			(justify right)
-		)
-		(property "Intersheetrefs" "${INTERSHEET_REFS}"
-			(at 14.7342 154.94 0)
-			(effects
-				(font
-					(size 1.27 1.27)
-				)
-				(justify right)
-				(hide yes)
-			)
-		)
-	)
 	(global_label "XSHUT_LEFT"
 		(shape input)
@@
 			(effects
 				(font
-					(size 1.27 1.27)
-				)
-				(justify right)
-				(hide yes)
-			)
-		)
-	)
-	(global_label "GPIOI_CENTER"
-		(shape input)
-		(at 29.21 172.72 180)
-		(fields_autoplaced yes)
-		(effects
-			(font
-				(size 1.27 1.27)
-			)
-			(justify right)
-		)
-		(property "Intersheetrefs" "${INTERSHEET_REFS}"
-			(at 13.041 172.72 0)
-			(effects
-				(font
