File: ECAD/Mini-PAMI-2025/Mini-PAMI-2025.kicad_pcb (KiCad board)
At the start: 2 copper layers, 52 x 52 mm, 14 parts, among them J1 Conn_01x05, J2 Conn_01x05, SW3 SW_Push, U2 MCP23008-xSO, U3 MOUDLE-SEEEDUINO-XIAO-ESP32C3, U4 AMS1117-5.0, U5 ULN2803A

Commit message: minor update
Parts:
- moved J2 2.88 mm to (54.0, 87.1)
- moved J1 2.05 mm to (54.0, 70.9)
- moved U2 1.63 mm to (81.3, 97.5)
- moved U3 0.19 mm to (66.3, 87.1)
Changed lines of the file:
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@@
 		(tags "SOIC SO")
 		(property "Reference" "U5"
-			(at 0 -6.72 360)
+			(at 0 -6.72 0)
 			(layer "F.SilkS")
 			(effects
@@
 		)
 		(property "Value" "ULN2803A"
-			(at 0 6.72 360)
+			(at 0 6.72 0)
 			(layer "F.Fab")
 			(effects
@@
 		)
 		(property "Footprint" "Package_SO:SOIC-18W_7.5x11.6mm_P1.27mm"
-			(at 0 0 360)
+			(at 0 0 0)
 			(layer "F.Fab")
 			(hide yes)
@@
 		)
 		(property "Datasheet" "http://www.ti.com/lit/ds/symlink/uln2803a.pdf"
-			(at 0 0 360)
+			(at 0 0 0)
 			(layer "F.Fab")
 			(hide yes)
@@
 		)
 		(property "Description" "Darlington Transistor Arrays, SOIC18/DIP18"
-			(at 0 0 360)
+			(at 0 0 0)
 			(layer "F.Fab")
 			(hide yes)
@@
 		)
 		(fp_text user "${REFERENCE}"
-			(at 0 0 360)
+			(at 0 0 0)
 			(layer "F.Fab")
 			(effects
@@
 	(footprint "Package_SO:SOIC-18W_7.5x11.6mm_P1.27mm"
 		(layer "F.Cu")
-		(at 82 99 180)
+		(at 81.28 97.536 180)
 		(descr "SOIC, 18 Pin (JEDEC MS-013AB, https://www.analog.com/media/en/package-pcb-resources/package/33254132129439rw_18.pdf), generated with kicad-footprint-generator ipc_gullwing_generator.py")
 		(tags "SOIC SO")
 		(property "Reference" "U2"
-			(at 0 -6.72 360)
+			(at 0 -6.72 0)
 			(layer "F.SilkS")
 			(effects
@@
 		)
 		(property "Value" "MCP23008-xSO"
-			(at 0 6.72 360)
+			(at 0 6.72 0)
 			(layer "F.Fab")
 			(effects
@@
 		)
 		(property "Footprint" "Package_SO:SOIC-18W_7.5x11.6mm_P1.27mm"
-			(at 0 0 360)
+			(at 0 0 0)
 			(layer "F.Fab")
 			(hide yes)
@@
 		)
 		(property "Datasheet" "http://ww1.microchip.com/downloads/en/DeviceDoc/MCP23008-MCP23S08-Data-Sheet-20001919F.pdf"
-			(at 0 0 360)
+			(at 0 0 0)
 			(layer "F.Fab")
 			(hide yes)
@@
 		)
 		(property "Description" "8-bit I/O expander, I2C, interrupts, SOIC-18"
-			(at 0 0 360)
+			(at 0 0 0)
 			(layer "F.Fab")
 			(hide yes)
@@
 		)
 		(fp_text user "${REFERENCE}"
-			(at 0 0 360)
+			(at 0 0 0)
 			(layer "F.Fab")
 			(effects
@@
 	(footprint "xiao ESP32C3_PCB:MOUDLE14P-SMD-2.54-21X17.8MM"
 		(layer "F.Cu")
-		(at 66.0825 87.11925)
+		(at 66.2665 87.06525)
 		(property "Reference" "U3"
 			(at 9.3345 -21.7805 0)
@@
 			(polygon
 				(pts
-					(xy 69.067 74.35575) (xy 71.988 74.35575) (xy 71.988 76.38775) (xy 69.067 76.38775)
+					(xy 69.251 74.30175) (xy 72.172 74.30175) (xy 72.172 76.33375) (xy 69.251 76.33375)
 				)
 			)
@@
 			(polygon
 				(pts
-					(xy 69.7655 66.03725) (xy 71.5435 66.03725) (xy 71.5435 68.70425) (xy 69.7655 68.70425)
+					(xy 69.9495 65.98325) (xy 71.7275 65.98325) (xy 71.7275 68.65025) (xy 69.9495 68.65025)
 				)
 			)
@@
 			(polygon
 				(pts
-					(xy 69.7655 70.10125) (xy 71.5435 70.10125) (xy 71.5435 72.76825) (xy 69.7655 72.76825)
+					(xy 69.9495 70.04725) (xy 71.7275 70.04725) (xy 71.7275 72.71425) (xy 69.9495 72.71425)
 				)
 			)
@@
 			(polygon
 				(pts
-					(xy 72.4325 66.79925) (xy 77.6395 66.79925) (xy 77.6395 73.78425) (xy 72.4325 73.78425)
+					(xy 72.6165 66.74525) (xy 77.8235 66.74525) (xy 77.8235 73.73025) (xy 72.6165 73.73025)
 				)
 			)
@@
 			(polygon
 				(pts
-					(xy 72.4325 83.94425) (xy 78.1475 83.94425) (xy 78.1475 86.48425) (xy 72.4325 86.48425)
+					(xy 72.6165 83.89025) (xy 78.3315 83.89025) (xy 78.3315 86.43025) (xy 72.6165 86.43025)
 				)
 			)
@@
 			(polygon
 				(pts
-					(xy 75.8615 75.81625) (xy 78.9095 75.81625) (xy 78.9095 78.86425) (xy 75.8615 78.86425)
+					(xy 76.0455 75.76225) (xy 79.0935 75.76225) (xy 79.0935 78.81025) (xy 76.0455 78.81025)
 				)
 			)
@@
 			(polygon
 				(pts
-					(xy 78.4015 66.03725) (xy 80.1795 66.03725) (xy 80.1795 68.70425) (xy 78.4015 68.70425)
+					(xy 78.5855 65.98325) (xy 80.3635 65.98325) (xy 80.3635 68.65025) (xy 78.5855 68.65025)
 				)
 			)
@@
 			(polygon
 				(pts
-					(xy 78.4015 70.10125) (xy 80.1795 70.10125) (xy 80.1795 72.76825) (xy 78.4015 72.76825)
+					(xy 78.5855 70.04725) (xy 80.3635 70.04725) (xy 80.3635 72.71425) (xy 78.5855 72.71425)
 				)
 			)
@@
 	(footprint "Connector_JST:JST_XH_B5B-XH-A_1x05_P2.50mm_Vertical"
 		(layer "B.Cu")
-		(at 54 90 -90)
+		(at 54 87.122 -90)
 		(descr "JST XH series connector, B5B-XH-A (http://www.jst-mfg.com/product/pdf/eng/eXH.pdf), generated with kicad-footprint-generator")
 		(tags "connector JST XH vertical")
@@
 	(footprint "Connector_JST:JST_XH_B5B-XH-A_1x05_P2.50mm_Vertical"
 		(layer "B.Cu")
-		(at 54 73 -90)
+		(at 54 70.946 -90)
 		(descr "JST XH series connector, B5B-XH-A (http://www.jst-mfg.com/product/pdf/eng/eXH.pdf), generated with kicad-footprint-generator")
 		(tags "connector JST XH vertical")
@@
 		(layer "Edge.Cuts")
 	)
+	(dimension
+		(type aligned)
+		(layer "F.Fab")
+		(pts
+			(xy 98 66) (xy 98 118)
+		)
+		(height -8.68)
+		(gr_text "52,0000 mm"
+			(at 105.53 92 90)
+			(layer "F.Fab")
+			(effects
+				(font
+					(size 1 1)
+					(thickness 0.15)
+				)
+			)
+		)
+		(format
+			(prefix "")
+			(suffix "")
+			(units 3)
+			(units_format 1)
+			(precision 4)
+		)
+		(style
+			(thickness 0.1)
+			(arrow_length 1.27)
+			(text_position_mode 0)
+			(extension_height 0.58642)
+			(extension_offset 0.5) keep_text_aligned)
+	)
+	(dimension
+		(type aligned)
+		(layer "F.Fab")
+		(pts
+			(xy 102 70) (xy 50 70)
+		)
+		(height 10.309999)
+		(gr_text "52,0000 mm"
+			(at 76 58.540001 0)
+			(layer "F.Fab")
+			(effects
+				(font
+					(size 1 1)
+					(thickness 0.15)
+				)
+			)
+		)
+		(format
+			(prefix "")
+			(suffix "")
+			(units 3)
+			(units_format 1)
+			(precision 4)
+		)
+		(style
+			(thickness 0.1)
+			(arrow_length 1.27)
+			(text_position_mode 0)
+			(extension_height 0.58642)
+			(extension_offset 0.5) keep_text_aligned)
+	)
 )
